File: pcb/Macro Pad.kicad_pcb (KiCad board)
At the start: 2 copper layers, 80 x 61.5 mm, 9 parts, among them SW1 SW_Push, SW2 SW_Push, SW3 SW_Push, SW4 SW_Push, SW5 SW_Push, SW6 SW_Push, SW7 SW_Push, SW8 SW_Push, U1 XIAO-RP2040-DIP

Commit message: Add files via upload
Routing:
- added copper zone on B.Cu, net GND
- added copper zone on F.Cu, net GND
Other:
- outline, holes or cut-outs redrawn
- board text added: "ETCPAD"
- board text added: "XIAO HERE!"
